File: button_control_small/btnsm_a_bit_larger.sch (EAGLE design)
At the start: 77 parts, among them IC1 LP298XS, IC2 MEGA8-AI, IC3 FM24-SG, J1 AVR_SPI_PROG_3X2NS, J2 OUT-, J3 OUT+, Q1 310mA/60V/1.6Ω, Q2 4.3A/20V/54mΩ, Q3 4.3A/20V/54mΩ, Q4 310mA/60V/1.6Ω, Q5 4.3A/20V/54mΩ, Q6 3.6864MHz, T1 BC848, T2 BC848, T3 BC848, T4 BC848, T5 BC848, U1 ACS711ELCTR-25AB-T, U2 HC_05, U3 DS18B20

Commit message: Added extra ADC channels, filters to ADC & AREF
Switched to 4 layers board in order to have proper AGND and shield ADC channels from any noise.
Parts:
- removed 3V3_CONST: 3V_SW, wirepad:WIREPADSMD1,27-254
- removed C13: 10n, resistor:C-EUC0402
- removed C5: 100n, resistor:C-EUC0402
- added 4.2: 4.2, wirepad:WIREPADSMD1,27-254
- added 8.4: 8.4, wirepad:WIREPADSMD1,27-254
- added C18: 100n, resistor:C-EUC0402
- added C19, C20, C21, C22: 10n, resistor:C-EUC0402
- added L1: 10UH-225MA, Seeed-Inductor:SMD-INDUCTOR-10UH-225MA-10%(0806)
- added Q10, Q11, Q9: 310mA/60V/1.6Ω, SparkFun-DiscreteSemi:MOSFET-NCH-2N7002PW
- added Q7, Q8: 4.3A/20V/54mΩ, SparkFun-DiscreteSemi:MOSFET_PCH-IRLML2244
- added R29, R30, R35, R38, R40, R41, R45, R49: 100k, rcl:R-EU_R0402
- added R33, R36, R37, R43, R44: 100k 1%, SparkFun-Resistors:RESISTOR0805
- added R34: 200k 1%, SparkFun-Resistors:RESISTOR0805
- added R39: 250k 1%, SparkFun-Resistors:RESISTOR0805
- added R42: 1k, rcl:R-EU_R0402
- added R46: 1.2k 1%, SparkFun-Resistors:RESISTOR0805
- added R47: 6.2k 1%, SparkFun-Resistors:RESISTOR0805
- added R48: 200, rcl:R-EU_R0402
- added SUPPLY7: 2PT_GND_TIE, SparkFun-PowerSymbols:2PT_GND_TIE
- added U5: TL431BQDBZR, TL431BQDBZR:TL431BQDBZR
- C1: value 100n -> 10n; device resistor:C-EUC0603K -> resistor:C-EUC0402
- R2: value 282k -> 100k 1%; device rcl:R-EU_R0402 -> SparkFun-Resistors:RESISTOR0805
- R4: value 100k -> 200k 1%; device rcl:R-EU_R0402 -> SparkFun-Resistors:RESISTOR0805
Connections:
- removed net MOSI: IC2.PB3(MOSI/OC2), J1.4
- removed net PC0: IC2.PC0(ADC0), Q2.G, R28.1
- removed net PC1: C1.1, IC2.PC1(ADC1)
- removed net PC2: IC2.PC2(ADC2), R19.2
- removed net PWR_MEASURE_VCC: Q2.D, U1.VCC
- removed net SCK: IC2.PB5(SCK), J1.3
- new net ADC0: R29.2, R36.2, R39.2
- new net ADC1: R30.2, R33.2, R34.1
- new net ADC2: R2.1, R4.2, R40.2
- new net AGND: C1.2, C14.2, C19.2, C20.2, C21.2, C22.2, C4.2, R33.1, R36.1, R4.1, R43.1, R47.1, SUPPLY7.P$2, U5.ANODE
- new net AVCC: C4.1, IC2.AVCC, L1.2
- new net N$10: 8.4.P, Q7.S, R35.2
- new net N$12: 4.2.P, Q8.S, R38.2
- new net N$14: Q2.D, R44.2, R48.2, U1.VCC
- new net N$19: Q10.G, Q11.G, Q9.G, R42.1
- new net N$25: R46.2, R48.1
- new net N$26: IC3.WP, R49.1
- new net N$3: Q11.D, Q7.G, R35.1
- new net N$5: Q7.D, R34.2
- new net N$6: Q10.D, Q8.G, R38.1
- new net N$7: Q8.D, R2.2
- new net N$8: R37.1, R39.1
- new net PB3/MOSI: IC2.PB3(MOSI/OC2), J1.4, U1.FAULT#
- new net PB5/SCK: IC2.PB5(SCK), J1.3, R19.2, R42.2
- new net REF: R46.1, R47.2, U5.REF
- new net _A0: C19.1, IC2.PC0(ADC0), R29.1
- new net _A1: C20.1, IC2.PC1(ADC1), R30.1
- new net _A2: C21.1, IC2.PC2(ADC2), R40.1
- new net _A6: C1.1, IC2.ADC6, R45.1
- new net _A7: C22.1, IC2.ADC7, R41.1
- net ADC6: now also R43.2, R44.1, R45.2; no longer IC2.ADC6, U1.VOUT
- net ADC7: now also R41.2, U1.VOUT; no longer IC2.ADC7, R2.2, R4.1
- net AREF: now also U5.CATHODE; no longer C5.2
- net GND: now also C18.2, Q10.S, Q11.S, Q9.S, R49.2, SUPPLY7.P$1; no longer C13.2, C14.2, C4.2, C5.1, R4.2
- net N$11: now also Q9.D; no longer C1.2
- net N$23: now also R37.2; no longer R2.1
- net PB4/MISO: now also Q2.G, R28.1; no longer R5.2
- net VCC: now also R1.2, R5.2
- net VDD: now also C18.1, L1.1; no longer 3V3_CONST.P, C13.1, C4.1, IC2.AVCC, R1.2
Other:
- note removed: "Вход с МК - включение измерителя"
- note removed: "Выход на МК - можно без прерывания"
- note removed: "в выходу мк, который управляем активацией АЦП должны быть импульсы по примерно 2мс"
- moved on the sheet: 3V3_SWITCHED, C1, C11, C7, C8, IC1, PAD2, Q1, Q5, R1, R10, R19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

Commit message: Bump to 5.8
Parts:
- added R50, R51: 6.2k 1%, SparkFun-Resistors:RESISTOR0805
- R37: value 100k 1% -> 120k 1%
- R39: value 250k 1% -> 270k 1%
- renumbered 3V3_SWITCHED to 3V3
Connections:
- removed net N$25: R46.2, R48.1
- net AREF: now also R46.2, R48.1
- net SCL: now also R50.1
- net SDA: now also R51.1
- net VCC: now also R50.2, R51.2
Changed lines of the file:
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@@
 <part name="PAD2" library="wirepad" library_urn="urn:adsk.eagle:library:412" deviceset="WIREPAD" device="SMD1,27-254" package3d_urn="urn:adsk.eagle:package:30839/1" value="WTR_IN"/>
 <part name="SUPPLY4" library="SparkFun-PowerSymbols" library_urn="urn:adsk.eagle:library:530" deviceset="VCC" device=""/>
-<part name="3V3_SWITCHED" library="wirepad" library_urn="urn:adsk.eagle:library:412" deviceset="WIREPAD" device="SMD1,27-254" package3d_urn="urn:adsk.eagle:package:30839/1" value="3V3"/>
+<part name="3V3" library="wirepad" library_urn="urn:adsk.eagle:library:412" deviceset="WIREPAD" device="SMD1,27-254" package3d_urn="urn:adsk.eagle:package:30839/1" value="3V3"/>
 <part name="IC1" library="adafruit" library_urn="urn:adsk.eagle:library:420" deviceset="LP298X" device="S"/>
 <part name="C11" library="resistor" library_urn="urn:adsk.eagle:library:348" deviceset="C-EU" device="C0402" package3d_urn="urn:adsk.eagle:package:26136/1" value="10n"/>
@@
 <part name="Q8" library="SparkFun-DiscreteSemi" library_urn="urn:adsk.eagle:library:514" deviceset="MOSFET_PCH" device="-IRLML2244" package3d_urn="urn:adsk.eagle:package:38446/1" value="4.3A/20V/54mΩ"/>
 <part name="R38" library="rcl" library_urn="urn:adsk.eagle:library:334" deviceset="R-EU_" device="R0402" package3d_urn="urn:adsk.eagle:package:23547/2" value="100k"/>
-<part name="R39" library="SparkFun-Resistors" library_urn="urn:adsk.eagle:library:532" deviceset="RESISTOR" device="0805" package3d_urn="urn:adsk.eagle:package:39651/1" value="250k 1%"/>
+<part name="R39" library="SparkFun-Resistors" library_urn="urn:adsk.eagle:library:532" deviceset="RESISTOR" device="0805" package3d_urn="urn:adsk.eagle:package:39651/1" value="270k 1%"/>
 <part name="R2" library="SparkFun-Resistors" library_urn="urn:adsk.eagle:library:532" deviceset="RESISTOR" device="0805" package3d_urn="urn:adsk.eagle:package:39651/1" value="100k 1%"/>
 <part name="R4" library="SparkFun-Resistors" library_urn="urn:adsk.eagle:library:532" deviceset="RESISTOR" device="0805" package3d_urn="urn:adsk.eagle:package:39651/1" value="200k 1%"/>
@@
 <part name="R34" library="SparkFun-Resistors" library_urn="urn:adsk.eagle:library:532" deviceset="RESISTOR" device="0805" package3d_urn="urn:adsk.eagle:package:39651/1" value="200k 1%"/>
 <part name="R36" library="SparkFun-Resistors" library_urn="urn:adsk.eagle:library:532" deviceset="RESISTOR" device="0805" package3d_urn="urn:adsk.eagle:package:39651/1" value="100k 1%"/>
-<part name="R37" library="SparkFun-Resistors" library_urn="urn:adsk.eagle:library:532" deviceset="RESISTOR" device="0805" package3d_urn="urn:adsk.eagle:package:39651/1" value="100k 1%"/>
+<part name="R37" library="SparkFun-Resistors" library_urn="urn:adsk.eagle:library:532" deviceset="RESISTOR" device="0805" package3d_urn="urn:adsk.eagle:package:39651/1" value="120k 1%"/>
 <part name="4.2" library="wirepad" library_urn="urn:adsk.eagle:library:412" deviceset="WIREPAD" device="SMD1,27-254" package3d_urn="urn:adsk.eagle:package:30839/1" value="4.2"/>
 <part name="8.4" library="wirepad" library_urn="urn:adsk.eagle:library:412" deviceset="WIREPAD" device="SMD1,27-254" package3d_urn="urn:adsk.eagle:package:30839/1" value="8.4"/>
@@
 <part name="GND33" library="supply1" library_urn="urn:adsk.eagle:library:371" deviceset="GND" device=""/>
 <part name="R49" library="rcl" library_urn="urn:adsk.eagle:library:334" deviceset="R-EU_" device="R0402" package3d_urn="urn:adsk.eagle:package:23547/2" value="100k"/>
+<part name="R50" library="SparkFun-Resistors" library_urn="urn:adsk.eagle:library:532" deviceset="RESISTOR" device="0805" package3d_urn="urn:adsk.eagle:package:39651/1" value="6.2k 1%"/>
+<part name="R51" library="SparkFun-Resistors" library_urn="urn:adsk.eagle:library:532" deviceset="RESISTOR" device="0805" package3d_urn="urn:adsk.eagle:package:39651/1" value="6.2k 1%"/>
+<part name="SUPPLY8" library="SparkFun-PowerSymbols" library_urn="urn:adsk.eagle:library:530" deviceset="VCC" device=""/>
+<part name="SUPPLY9" library="SparkFun-PowerSymbols" library_urn="urn:adsk.eagle:library:530" deviceset="VCC" device=""/>
 </parts>
 <sheets>
@@
 <instance part="PAD2" gate="G$1" x="231.14" y="261.62" rot="R180"/>
 <instance part="SUPPLY4" gate="G$1" x="180.34" y="281.94"/>
-<instance part="3V3_SWITCHED" gate="G$1" x="172.72" y="276.86"/>
+<instance part="3V3" gate="G$1" x="172.72" y="276.86"/>
 <instance part="IC1" gate="G$1" x="0" y="-25.4" rot="R270"/>
 <instance part="C11" gate="G$1" x="12.7" y="-33.02"/>
@@
 <instance part="GND33" gate="1" x="266.7" y="88.9" rot="MR0"/>
 <instance part="R49" gate="G$1" x="266.7" y="99.06" rot="MR270"/>
+<instance part="R50" gate="G$1" x="269.24" y="116.84" rot="R90"/>
+<instance part="R51" gate="G$1" x="317.5" y="116.84" rot="R90"/>
+<instance part="SUPPLY8" gate="G$1" x="269.24" y="124.46"/>
+<instance part="SUPPLY9" gate="G$1" x="317.5" y="124.46"/>
 </instances>
 <busses>
@@
 <segment>
 <pinref part="U5" gate="A" pin="CATHODE"/>
-<wire x1="434.34" y1="203.2" x2="452.12" y2="203.2" width="0.1524" layer="91"/>
+<wire x1="434.34" y1="203.2" x2="441.96" y2="203.2" width="0.1524" layer="91"/>
 <label x="444.5" y="203.2" size="1.778" layer="95"/>
+<pinref part="R48" gate="G$1" pin="1"/>
+<pinref part="R46" gate="G$1" pin="2"/>
+<wire x1="441.96" y1="203.2" x2="452.12" y2="203.2" width="0.1524" layer="91"/>
+<wire x1="373.38" y1="218.44" x2="386.08" y2="218.44" width="0.1524" layer="91"/>
+<wire x1="386.08" y1="218.44" x2="441.96" y2="218.44" width="0.1524" layer="91"/>
+<wire x1="441.96" y1="218.44" x2="441.96" y2="203.2" width="0.1524" layer="91"/>
+<junction x="386.08" y="218.44"/>
+<junction x="441.96" y="203.2"/>
 </segment>
 <segment>
@@
 <wire x1="180.34" y1="276.86" x2="180.34" y2="271.78" width="0.1524" layer="91"/>
 <wire x1="180.34" y1="281.94" x2="180.34" y2="279.4" width="0.1524" layer="91"/>
-<pinref part="3V3_SWITCHED" gate="G$1" pin="P"/>
+<pinref part="3V3" gate="G$1" pin="P"/>
 <wire x1="175.26" y1="276.86" x2="180.34" y2="276.86" width="0.1524" layer="91"/>
 <junction x="180.34" y="276.86"/>
@@
 <pinref part="SUPPLY6" gate="G$1" pin="VCC"/>
 <wire x1="132.08" y1="236.22" x2="132.08" y2="228.6" width="0.1524" layer="91"/>
+</segment>
+<segment>
+<pinref part="SUPPLY8" gate="G$1" pin="VCC"/>
+<pinref part="R50" gate="G$1" pin="2"/>
+<wire x1="269.24" y1="124.46" x2="269.24" y2="121.92" width="0.1524" layer="91"/>
+</segment>
+<segment>
+<pinref part="SUPPLY9" gate="G$1" pin="VCC"/>
+<pinref part="R51" gate="G$1" pin="2"/>
+<wire x1="317.5" y1="124.46" x2="317.5" y2="121.92" width="0.1524" layer="91"/>
 </segment>
 </net>
@@
 <segment>
 <pinref part="IC3" gate="G$1" pin="SDA"/>
-<wire x1="307.34" y1="99.06" x2="320.04" y2="99.06" width="0.1524" layer="91"/>
+<wire x1="307.34" y1="99.06" x2="317.5" y2="99.06" width="0.1524" layer="91"/>
 <label x="309.88" y="99.06" size="1.778" layer="95"/>
+<pinref part="R51" gate="G$1" pin="1"/>
+<wire x1="317.5" y1="99.06" x2="320.04" y2="99.06" width="0.1524" layer="91"/>
+<wire x1="317.5" y1="111.76" x2="317.5" y2="99.06" width="0.1524" layer="91"/>
+<junction x="317.5" y="99.06"/>
 </segment>
 </net>
@@
 <segment>
 <pinref part="IC3" gate="G$1" pin="SCL"/>
-<wire x1="274.32" y1="106.68" x2="261.62" y2="106.68" width="0.1524" layer="91"/>
+<wire x1="274.32" y1="106.68" x2="269.24" y2="106.68" width="0.1524" layer="91"/>
 <label x="264.16" y="106.68" size="1.778" layer="95"/>
+<pinref part="R50" gate="G$1" pin="1"/>
+<wire x1="269.24" y1="106.68" x2="261.62" y2="106.68" width="0.1524" layer="91"/>
+<wire x1="269.24" y1="111.76" x2="269.24" y2="106.68" width="0.1524" layer="91"/>
+<junction x="269.24" y="106.68"/>
 </segment>
 </net>
@@
 </segment>
 </net>
-<net name="N$25" class="0">
-<segment>
-<pinref part="R48" gate="G$1" pin="1"/>
-<pinref part="R46" gate="G$1" pin="2"/>
-<wire x1="373.38" y1="218.44" x2="386.08" y2="218.44" width="0.1524" layer="91"/>
-</segment>
-</net>
